Commit message: add remotes

File: john_deere.urdf (robot description, URDF)
Before this commit: robot kubo, 121 links, 120 joints
Links:
- link ark_cam_mini_bracket_front: geometry collision box size=0.05 0.05 0.05; visual mesh filename=file:///home/ros/ws/common_ws/install/sensor_description/sh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 scale=0.001 0.001 0.001
- link ark_cam_mini_bracket_rear: geometry collision box size=0.05 0.05 0.05; visual mesh filename=file:///home/ros/ws/common_ws/install/sensor_description/sh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 scale=0.001 0.001 0.001
- link implement_camera_bracket_front_left: geometry collision box size=0.05 0.05 0.05; visual mesh filename=file:///home/ros/ws/common_ws/install/sensor_description/sh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 scale=0.001 0.001 0.001
- link implement_camera_bracket_front_right: geometry collision box size=0.05 0.05 0.05; visual mesh filename=file:///home/ros/ws/common_ws/install/sensor_description/sh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 scale=0.001 0.001 0.001
- link implement_camera_bracket_rear: geometry collision box size=0.05 0.05 0.05; visual mesh filename=file:///home/ros/ws/common_ws/install/sensor_description/sh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 scale=0.001 0.001 0.001
- link implement_radar_camera_bracket_front_left: geometry collision box size=0.05 0.05 0.05; visual mesh filename=file:///home/ros/ws/common_ws/install/sensor_description/sh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 scale=0.001 0.001 0.001
- link implement_radar_camera_bracket_front_right: geometry collision box size=0.05 0.05 0.05; visual mesh filename=file:///home/ros/ws/common_ws/install/sensor_description/sh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 scale=0.001 0.001 0.001
- link implement_radar_camera_bracket_rear: geometry collision box size=0.05 0.05 0.05; visual mesh filename=file:///home/ros/ws/common_ws/install/sensor_description/sh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 scale=0.001 0.001 0.001
- link nominal_implement_camera_mount_front_left: geometry collision mesh filename=file:///home/ros/ws/common_ws/install/sensor_description/sh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 scale=0.001 0.001 0.001; visual mesh filename=file:///home/ros/ws/common_ws/install/sensor_description/sh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 scale=0.001 0.001 0.001
- link nominal_implement_camera_mount_front_right: geometry collision mesh filename=file:///home/ros/ws/common_ws/install/sensor_description/sh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 scale=0.001 0.001 0.001; visual mesh filename=file:///home/ros/ws/common_ws/install/sensor_description/sh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 scale=0.001 0.001 0.001
- link nominal_implement_camera_mount_rear: geometry collision mesh filename=file:///home/ros/ws/common_ws/install/sensor_description/sh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 scale=0.001 0.001 0.001; visual mesh filename=file:///home/ros/ws/common_ws/install/sensor_description/sh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 scale=0.001 0.001 0.001
- link nominal_implement_radar_front_left: geometry collision box size=0.02 0.1 0.1; visual mesh filename=file:///home/ros/ws/common_ws/install/sensor_description/sh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 scale=1.0 1.0 1.0
- link nominal_implement_radar_front_right: geometry collision box size=0.02 0.1 0.1; visual mesh filename=file:///home/ros/ws/common_ws/install/sensor_description/sh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 scale=1.0 1.0 1.0
- link nominal_implement_radar_rear: geometry collision box size=0.02 0.1 0.1; visual mesh filename=file:///home/ros/ws/common_ws/install/sensor_description/sh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 scale=1.0 1.0 1.0
- link nominal_tractor_camera_bracket_middle_left: geometry collision box size=0.05 0.05 0.05; visual mesh filename=file:///home/ros/ws/common_ws/install/sensor_description/sh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 scale=0.001 0.001 0.001
- link nominal_tractor_camera_bracket_middle_right: geometry collision box size=0.05 0.05 0.05; visual mesh filename=file:///home/ros/ws/common_ws/install/sensor_description/sh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 scale=0.001 0.001 0.001
- link nominal_tractor_camera_mount_front: geometry collision mesh filename=file:///home/ros/ws/common_ws/install/sensor_description/sh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 scale=0.001 0.001 0.001; visual mesh filename=file:///home/ros/ws/common_ws/install/sensor_description/sh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 scale=0.001 0.001 0.001
- link nominal_tractor_camera_mount_middle_left: geometry collision mesh filename=file:///home/ros/ws/common_ws/install/sensor_description/sh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 scale=0.001 0.001 0.001; visual mesh filename=file:///home/ros/ws/common_ws/install/sensor_description/sh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 scale=0.001 0.001 0.001
- link nominal_tractor_camera_mount_middle_right: geometry collision mesh filename=file:///home/ros/ws/common_ws/install/sensor_description/sh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 scale=0.001 0.001 0.001; visual mesh filename=file:///home/ros/ws/common_ws/install/sensor_description/sh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 scale=0.001 0.001 0.001
- link nominal_tractor_camera_mount_rear: geometry collision mesh filename=file:///home/ros/ws/common_ws/install/sensor_description/sh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 scale=0.001 0.001 0.001; visual mesh filename=file:///home/ros/ws/common_ws/install/sensor_description/sh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 scale=0.001 0.001 0.001

File: john_deere_copy.urdf (robot description, URDF)
Before this commit: robot kubo, 121 links, 120 joints
Links:
- link ark_cam_mini_bracket_front: geometry collision box size=0.05 0.05 0.05; visual mesh filename=file:///home/ros/ws/atemp_ws/urdf-test/meshes/ark_cam_basic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 scale=0.001 0.001 0.001
- link ark_cam_mini_bracket_rear: geometry collision box size=0.05 0.05 0.05; visual mesh filename=file:///home/ros/ws/atemp_ws/urdf-test/meshes/ark_cam_basic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 scale=0.001 0.001 0.001
- link cover: geometry collision mesh filename=file:///home/ros/ws/atemp_ws/urdf-test/meshes/JD6M.dae; visual mesh filename=file:///home/ros/ws/atemp_ws/urdf-test/meshes/JD6M.dae
- link implement_base: geometry collision mesh filename=file:///home/ros/ws/atemp_ws/urdf-test/meshes/lemken_karat_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 scale=1.0 1.0 1.0; visual mesh filename=file:///home/ros/ws/atemp_ws/urdf-test/meshes/lemken_karat_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 scale=1.0 1.0 1.0
- link implement_camera_bracket_front_left: geometry collision box size=0.05 0.05 0.05; visual mesh filename=file:///home/ros/ws/atemp_ws/urdf-test/meshes/ark_cam_basic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 scale=0.001 0.001 0.001
- link implement_camera_bracket_front_right: geometry collision box size=0.05 0.05 0.05; visual mesh filename=file:///home/ros/ws/atemp_ws/urdf-test/meshes/ark_cam_basic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 scale=0.001 0.001 0.001
- link implement_camera_bracket_rear: geometry collision box size=0.05 0.05 0.05; visual mesh filename=file:///home/ros/ws/atemp_ws/urdf-test/meshes/ark_cam_basic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 scale=0.001 0.001 0.001
- link implement_radar_camera_bracket_front_left: geometry collision box size=0.05 0.05 0.05; visual mesh filename=file:///home/ros/ws/atemp_ws/urdf-test/meshes/radar_camera_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 scale=0.001 0.001 0.001
- link implement_radar_camera_bracket_front_right: geometry collision box size=0.05 0.05 0.05; visual mesh filename=file:///home/ros/ws/atemp_ws/urdf-test/meshes/radar_camera_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 scale=0.001 0.001 0.001
- link implement_radar_camera_bracket_rear: geometry collision box size=0.05 0.05 0.05; visual mesh filename=file:///home/ros/ws/atemp_ws/urdf-test/meshes/radar_camera_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 scale=0.001 0.001 0.001
- link left_front_wheel: geometry collision cylinder length=0.1 radius=0.7135; visual mesh filename=file:///home/ros/ws/atemp_ws/urdf-test/meshes/front_wheel.d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 scale=1.9819444444444445 2.938888888888889 1.9819444444444445
- link left_rear_wheel: geometry collision cylinder length=0.1 radius=0.945; visual mesh filename=file:///home/ros/ws/atemp_ws/urdf-test/meshes/rear_wheel.dae scale=2.5 3.588888888888889 2.5
- link nominal_implement_camera_mount_front_left: geometry collision mesh filename=file:///home/ros/ws/atemp_ws/urdf-test/meshes/ark_cam_basic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 scale=0.001 0.001 0.001; visual mesh filename=file:///home/ros/ws/atemp_ws/urdf-test/meshes/ark_cam_basic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 scale=0.001 0.001 0.001
- link nominal_implement_camera_mount_front_right: geometry collision mesh filename=file:///home/ros/ws/atemp_ws/urdf-test/meshes/ark_cam_basic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 scale=0.001 0.001 0.001; visual mesh filename=file:///home/ros/ws/atemp_ws/urdf-test/meshes/ark_cam_basic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 scale=0.001 0.001 0.001
- link nominal_implement_camera_mount_rear: geometry collision mesh filename=file:///home/ros/ws/atemp_ws/urdf-test/meshes/ark_cam_basic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 scale=0.001 0.001 0.001; visual mesh filename=file:///home/ros/ws/atemp_ws/urdf-test/meshes/ark_cam_basic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 scale=0.001 0.001 0.001
- link nominal_implement_lidar_front: geometry collision cylinder length=0.0717 radius=0.0516; visual mesh filename=file:///home/ros/ws/atemp_ws/urdf-test/meshes/OS0.dae
- link nominal_implement_radar_front_left: geometry collision box size=0.02 0.1 0.1; visual mesh filename=file:///home/ros/ws/atemp_ws/urdf-test/meshes/smartmicro_ty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 scale=1.0 1.0 1.0
- link nominal_implement_radar_front_right: geometry collision box size=0.02 0.1 0.1; visual mesh filename=file:///home/ros/ws/atemp_ws/urdf-test/meshes/smartmicro_ty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 scale=1.0 1.0 1.0
- link nominal_implement_radar_rear: geometry collision box size=0.02 0.1 0.1; visual mesh filename=file:///home/ros/ws/atemp_ws/urdf-test/meshes/smartmicro_ty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 scale=1.0 1.0 1.0
- link nominal_implement_stereo_zed2x_rear: geometry collision box size=0.02 0.1 0.1; visual mesh filename=file:///home/ros/ws/atemp_ws/urdf-test/meshes/zed2i.stl scale=1 1 1
- link nominal_tractor_camera_bracket_middle_left: geometry collision box size=0.05 0.05 0.05; visual mesh filename=file:///home/ros/ws/atemp_ws/urdf-test/meshes/ark_cam_basic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 scale=0.001 0.001 0.001
- link nominal_tractor_camera_bracket_middle_right: geometry collision box size=0.05 0.05 0.05; visual mesh filename=file:///home/ros/ws/atemp_ws/urdf-test/meshes/ark_cam_basic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 scale=0.001 0.001 0.001
- link nominal_tractor_camera_mount_front: geometry collision mesh filename=file:///home/ros/ws/atemp_ws/urdf-test/meshes/ark_cam_basic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 scale=0.001 0.001 0.001; visual mesh filename=file:///home/ros/ws/atemp_ws/urdf-test/meshes/ark_cam_basic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 scale=0.001 0.001 0.001
- link nominal_tractor_camera_mount_middle_left: geometry collision mesh filename=file:///home/ros/ws/atemp_ws/urdf-test/meshes/ark_cam_basic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 scale=0.001 0.001 0.001; visual mesh filename=file:///home/ros/ws/atemp_ws/urdf-test/meshes/ark_cam_basic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 scale=0.001 0.001 0.001
- link nominal_tractor_camera_mount_middle_right: geometry collision mesh filename=file:///home/ros/ws/atemp_ws/urdf-test/meshes/ark_cam_basic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 scale=0.001 0.001 0.001; visual mesh filename=file:///home/ros/ws/atemp_ws/urdf-test/meshes/ark_cam_basic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 scale=0.001 0.001 0.001
- link nominal_tractor_camera_mount_rear: geometry collision mesh filename=file:///home/ros/ws/atemp_ws/urdf-test/meshes/ark_cam_basic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 scale=0.001 0.001 0.001; visual mesh filename=file:///home/ros/ws/atemp_ws/urdf-test/meshes/ark_cam_basic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 scale=0.001 0.001 0.001
- link nominal_tractor_lidar_front: geometry collision cylinder length=0.0717 radius=0.0516; visual mesh filename=file:///home/ros/ws/atemp_ws/urdf-test/meshes/OS0.dae
- link nominal_tractor_lidar_rear: geometry collision cylinder length=0.0717 radius=0.0516; visual mesh filename=file:///home/ros/ws/atemp_ws/urdf-test/meshes/OS0.dae
- link nominal_tractor_radar_front_left: geometry collision box size=0.02 0.1 0.1; visual mesh filename=file:///home/ros/ws/atemp_ws/urdf-test/meshes/smartmicro_ty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 scale=1.0 1.0 1.0
- link nominal_tractor_radar_front_right: geometry collision box size=0.02 0.1 0.1; visual mesh filename=file:///home/ros/ws/atemp_ws/urdf-test/meshes/smartmicro_ty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 scale=1.0 1.0 1.0
- link nominal_tractor_radar_middle_left: geometry collision box size=0.02 0.1 0.1; visual mesh filename=file:///home/ros/ws/atemp_ws/urdf-test/meshes/smartmicro_ty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 scale=1.0 1.0 1.0
- link nominal_tractor_radar_middle_right: geometry collision box size=0.02 0.1 0.1; visual mesh filename=file:///home/ros/ws/atemp_ws/urdf-test/meshes/smartmicro_ty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 scale=1.0 1.0 1.0
- link right_front_wheel: geometry collision cylinder length=0.1 radius=0.7135; visual mesh filename=file:///home/ros/ws/atemp_ws/urdf-test/meshes/front_wheel.d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 scale=1.9819444444444445 2.938888888888889 1.9819444444444445
- link right_rear_wheel: geometry collision cylinder length=0.1 radius=0.945; visual mesh filename=file:///home/ros/ws/atemp_ws/urdf-test/meshes/rear_wheel.dae scale=2.5 3.588888888888889 2.5
- link tractor_gnss_autotrac_link: geometry collision cylinder length=0.05 radius=0.1; visual mesh filename=file:///home/ros/ws/atemp_ws/urdf-test/meshes/generic_gnss.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
- link tractor_gnss_left_mount: geometry collision cylinder length=0.05 radius=0.1; visual mesh filename=file:///home/ros/ws/atemp_ws/urdf-test/meshes/smart7.stl scale=0.001 0.001 0.001
- link tractor_gnss_right_mount: geometry collision cylinder length=0.05 radius=0.1; visual mesh filename=file:///home/ros/ws/atemp_ws/urdf-test/meshes/smart7.stl scale=0.001 0.001 0.001
