Commit message: update rd25 with saferadar frame

File: thorsen_fort_rd25.urdf (robot description, URDF)
Before this commit: robot fort_rd25, 27 links, 26 joints
Links:
- added link tractor_radar_saferadar, mass 0.0005
- link nominal_tractor_camera_mount_front: geometry collision mesh filename=package://sensor_description/models/arkvision_arkcam_mini/m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 scale=0.001 0.001 0.001; visual mesh filename=file:///home/ros/ws/common_ws/install/sensor_description/sh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 scale=0.001 0.001 0.001
- link nominal_tractor_camera_mount_rear: geometry collision mesh filename=package://sensor_description/models/arkvision_arkcam_mini/m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 scale=0.001 0.001 0.001; visual mesh filename=file:///home/ros/ws/common_ws/install/sensor_description/sh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 scale=0.001 0.001 0.001
- link tractor_imu_center: geometry collision box size=0.05 0.05 0.05; visual box size=0.05 0.05 0.05
Joints:
- added joint base_link_tractor_radar_saferadar_joint: type fixed, parent base_link, child tractor_radar_saferadar, origin xyz=0.98 0 1.175 rpy=0 0 0

File: thorsen_fort_rd25_remote.urdf (robot description, URDF)
Before this commit: robot fort_rd25, 27 links, 26 joints
Links:
- added link tractor_radar_saferadar, mass 0.0005
- link nominal_tractor_camera_mount_front: geometry collision mesh filename=package://sensor_description/models/arkvision_arkcam_mini/m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 scale=0.001 0.001 0.001; visual mesh filename=https://raw.githubusercontent.com/CM134/urdf-test/main/mesh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 scale=0.001 0.001 0.001
- link nominal_tractor_camera_mount_rear: geometry collision mesh filename=package://sensor_description/models/arkvision_arkcam_mini/m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 scale=0.001 0.001 0.001; visual mesh filename=https://raw.githubusercontent.com/CM134/urdf-test/main/mesh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 scale=0.001 0.001 0.001
- link tractor_imu_center: geometry collision box size=0.05 0.05 0.05; visual box size=0.05 0.05 0.05
Joints:
- added joint base_link_tractor_radar_saferadar_joint: type fixed, parent base_link, child tractor_radar_saferadar, origin xyz=0.98 0 1.175 rpy=0 0 0
