Commit message: update repo

File: urdf/lemken_john_deere_6r_SN-002-0001_lemken_karat_10_SN-003-0003_remote.urdf (robot description, URDF)
Before this commit: robot kubo, 121 links, 120 joints
Links:
- link ark_cam_mini_bracket_front: geometry collision box size=0.05 0.05 0.05; visual mesh filename=https://gitlab.com/agrirobot_public/remote_urdf/-/raw/main/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 scale=0.001 0.001 0.001
- link ark_cam_mini_bracket_rear: geometry collision box size=0.05 0.05 0.05; visual mesh filename=https://gitlab.com/agrirobot_public/remote_urdf/-/raw/main/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 scale=0.001 0.001 0.001
- link cover: geometry collision mesh filename=https://gitlab.com/agrirobot_public/remote_urdf/-/raw/main/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; visual mesh filename=https://gitlab.com/agrirobot_public/remote_urdf/-/raw/main/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
- link implement_base: geometry collision mesh filename=https://gitlab.com/agrirobot_public/remote_urdf/-/raw/main/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 scale=1.0 1.0 1.0; visual mesh filename=https://gitlab.com/agrirobot_public/remote_urdf/-/raw/main/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 scale=1.0 1.0 1.0
- link implement_camera_bracket_front_left: geometry collision box size=0.05 0.05 0.05; visual mesh filename=https://gitlab.com/agrirobot_public/remote_urdf/-/raw/main/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 scale=0.001 0.001 0.001
- link implement_camera_bracket_front_right: geometry collision box size=0.05 0.05 0.05; visual mesh filename=https://gitlab.com/agrirobot_public/remote_urdf/-/raw/main/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 scale=0.001 0.001 0.001
- link implement_camera_bracket_rear: geometry collision box size=0.05 0.05 0.05; visual mesh filename=https://gitlab.com/agrirobot_public/remote_urdf/-/raw/main/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 scale=0.001 0.001 0.001
- link implement_radar_camera_bracket_front_left: geometry collision box size=0.05 0.05 0.05; visual mesh filename=https://gitlab.com/agrirobot_public/remote_urdf/-/raw/main/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 scale=0.001 0.001 0.001
- link implement_radar_camera_bracket_front_right: geometry collision box size=0.05 0.05 0.05; visual mesh filename=https://gitlab.com/agrirobot_public/remote_urdf/-/raw/main/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 scale=0.001 0.001 0.001
- link implement_radar_camera_bracket_rear: geometry collision box size=0.05 0.05 0.05; visual mesh filename=https://gitlab.com/agrirobot_public/remote_urdf/-/raw/main/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 scale=0.001 0.001 0.001
- link left_front_wheel: geometry collision cylinder length=0.1 radius=0.7135; visual mesh filename=https://gitlab.com/agrirobot_public/remote_urdf/-/raw/main/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 scale=1.9819444444444445 2.938888888888889 1.9819444444444445
- link left_rear_wheel: geometry collision cylinder length=0.1 radius=0.945; visual mesh filename=https://gitlab.com/agrirobot_public/remote_urdf/-/raw/main/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 scale=2.5 3.588888888888889 2.5
- link nominal_implement_camera_mount_front_left: geometry collision mesh filename=https://gitlab.com/agrirobot_public/remote_urdf/-/raw/main/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 scale=0.001 0.001 0.001; visual mesh filename=https://gitlab.com/agrirobot_public/remote_urdf/-/raw/main/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 scale=0.001 0.001 0.001
- link nominal_implement_camera_mount_front_right: geometry collision mesh filename=https://gitlab.com/agrirobot_public/remote_urdf/-/raw/main/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 scale=0.001 0.001 0.001; visual mesh filename=https://gitlab.com/agrirobot_public/remote_urdf/-/raw/main/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 scale=0.001 0.001 0.001
- link nominal_implement_camera_mount_rear: geometry collision mesh filename=https://gitlab.com/agrirobot_public/remote_urdf/-/raw/main/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 scale=0.001 0.001 0.001; visual mesh filename=https://gitlab.com/agrirobot_public/remote_urdf/-/raw/main/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 scale=0.001 0.001 0.001
- link nominal_implement_lidar_front: geometry collision cylinder length=0.0717 radius=0.0516; visual mesh filename=https://gitlab.com/agrirobot_public/remote_urdf/-/raw/main/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
- link nominal_implement_radar_front_left: geometry collision box size=0.02 0.1 0.1; visual mesh filename=https://gitlab.com/agrirobot_public/remote_urdf/-/raw/main/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 scale=1.0 1.0 1.0
- link nominal_implement_radar_front_right: geometry collision box size=0.02 0.1 0.1; visual mesh filename=https://gitlab.com/agrirobot_public/remote_urdf/-/raw/main/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 scale=1.0 1.0 1.0
- link nominal_implement_radar_rear: geometry collision box size=0.02 0.1 0.1; visual mesh filename=https://gitlab.com/agrirobot_public/remote_urdf/-/raw/main/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 scale=1.0 1.0 1.0
- link nominal_implement_stereo_zed2x_rear: geometry collision box size=0.02 0.1 0.1; visual mesh filename=https://gitlab.com/agrirobot_public/remote_urdf/-/raw/main/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 scale=1 1 1
- link nominal_tractor_camera_bracket_middle_left: geometry collision box size=0.05 0.05 0.05; visual mesh filename=https://gitlab.com/agrirobot_public/remote_urdf/-/raw/main/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 scale=0.001 0.001 0.001
- link nominal_tractor_camera_bracket_middle_right: geometry collision box size=0.05 0.05 0.05; visual mesh filename=https://gitlab.com/agrirobot_public/remote_urdf/-/raw/main/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 scale=0.001 0.001 0.001
- link nominal_tractor_camera_mount_front: geometry collision mesh filename=https://gitlab.com/agrirobot_public/remote_urdf/-/raw/main/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 scale=0.001 0.001 0.001; visual mesh filename=https://gitlab.com/agrirobot_public/remote_urdf/-/raw/main/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 scale=0.001 0.001 0.001
- link nominal_tractor_camera_mount_middle_left: geometry collision mesh filename=https://gitlab.com/agrirobot_public/remote_urdf/-/raw/main/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 scale=0.001 0.001 0.001; visual mesh filename=https://gitlab.com/agrirobot_public/remote_urdf/-/raw/main/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 scale=0.001 0.001 0.001
- link nominal_tractor_camera_mount_middle_right: geometry collision mesh filename=https://gitlab.com/agrirobot_public/remote_urdf/-/raw/main/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 scale=0.001 0.001 0.001; visual mesh filename=https://gitlab.com/agrirobot_public/remote_urdf/-/raw/main/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 scale=0.001 0.001 0.001
- link nominal_tractor_camera_mount_rear: geometry collision mesh filename=https://gitlab.com/agrirobot_public/remote_urdf/-/raw/main/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 scale=0.001 0.001 0.001; visual mesh filename=https://gitlab.com/agrirobot_public/remote_urdf/-/raw/main/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 scale=0.001 0.001 0.001
- link nominal_tractor_lidar_front: geometry collision cylinder length=0.0717 radius=0.0516; visual mesh filename=https://gitlab.com/agrirobot_public/remote_urdf/-/raw/main/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
- link nominal_tractor_lidar_rear: geometry collision cylinder length=0.0717 radius=0.0516; visual mesh filename=https://gitlab.com/agrirobot_public/remote_urdf/-/raw/main/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
- link nominal_tractor_radar_front_left: geometry collision box size=0.02 0.1 0.1; visual mesh filename=https://gitlab.com/agrirobot_public/remote_urdf/-/raw/main/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 scale=1.0 1.0 1.0
- link nominal_tractor_radar_front_right: geometry collision box size=0.02 0.1 0.1; visual mesh filename=https://gitlab.com/agrirobot_public/remote_urdf/-/raw/main/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 scale=1.0 1.0 1.0
- link nominal_tractor_radar_middle_left: geometry collision box size=0.02 0.1 0.1; visual mesh filename=https://gitlab.com/agrirobot_public/remote_urdf/-/raw/main/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 scale=1.0 1.0 1.0
- link nominal_tractor_radar_middle_right: geometry collision box size=0.02 0.1 0.1; visual mesh filename=https://gitlab.com/agrirobot_public/remote_urdf/-/raw/main/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 scale=1.0 1.0 1.0
- link right_front_wheel: geometry collision cylinder length=0.1 radius=0.7135; visual mesh filename=https://gitlab.com/agrirobot_public/remote_urdf/-/raw/main/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 scale=1.9819444444444445 2.938888888888889 1.9819444444444445
- link right_rear_wheel: geometry collision cylinder length=0.1 radius=0.945; visual mesh filename=https://gitlab.com/agrirobot_public/remote_urdf/-/raw/main/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 scale=2.5 3.588888888888889 2.5
- link tractor_gnss_autotrac_link: geometry collision cylinder length=0.05 radius=0.1; visual mesh filename=https://gitlab.com/agrirobot_public/remote_urdf/-/raw/main/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
- link tractor_gnss_left_mount: geometry collision cylinder length=0.05 radius=0.1; visual mesh filename=https://gitlab.com/agrirobot_public/remote_urdf/-/raw/main/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 scale=0.001 0.001 0.001
- link tractor_gnss_right_mount: geometry collision cylinder length=0.05 radius=0.1; visual mesh filename=https://gitlab.com/agrirobot_public/remote_urdf/-/raw/main/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 scale=0.001 0.001 0.001
- link tractor_imu_center: geometry visual box size=0.05 0.05 0.05
Joints:
- joint base_link_to_chassis: origin xyz=0 0 1.0 rpy=0 -0.06 0 -> xyz=0 0 1.0 rpy=0 0 0
- joint nominal_implement_lidar_front_implement_lidar_front_joint: origin xyz=0.1 0 0 rpy=0 -0.09 3.14159265359 -> xyz=0.1 0 0 rpy=0 -0.1745 3.14159265359
- joint nominal_implement_radar_rear_implement_radar_rear_joint: origin xyz=0.1 0 0.3 rpy=0 0.7 0 -> xyz=0.1 0 0.3 rpy=0 0.576 0
- joint nominal_tractor_lidar_front_tractor_lidar_front_joint: origin xyz=0 0 0 rpy=-0.03 0 0 -> xyz=0 0 0 rpy=0 0 0
- joint nominal_tractor_lidar_rear_tractor_lidar_rear_joint: origin xyz=0 0 0 rpy=0 0.03 0 -> xyz=0 0 0 rpy=0 0 0
